File: kicad/emu1802_mini/emu1802_mini.kicad_pcb (KiCad board)
At the start: 2 copper layers, 47 x 72 mm, 25 parts, among them CON1 PICKIT/SNAP, CON2 UART, CON3 Software Serial, CON4 DC-IN, J1 CPUA, J2 CPUB, SW1 POWER, SW2 RESET, U1 CDP1802ACE, U2 PIC18F27Q43

Commit message: Updated emu1802-mini PCB Rev.1.0
Parts:
- added D2: 1N4148, Diode_THT:D_T-1_P5.08mm_Horizontal, F.Cu at (139.2, 113.7)
- added JP1: BUS POWER1, Jumper:SolderJumper-2_P1.3mm_Open_RoundedPad1.0x1.5mm, B.Cu at (112.5, 95.2)
- added JP2: BUS POWER2, Jumper:SolderJumper-2_P1.3mm_Open_RoundedPad1.0x1.5mm, B.Cu at (134.1, 111.1)
- moved C4 0.90 mm to (114.8, 99.7)
Connections:
- net Net-(CON4-Pad1) renamed +5V
- CON2 pad 3: unconnected-(CON2-Pad3) -> Net-(CON2-Pad3)
- CON3 pad 3: unconnected-(CON3-Pad3) -> Net-(CON3-Pad3)
- CON3 pad 4: /~EF3 -> Net-(CON3-Pad4)
Routing:
- net +5V: track 12.8 -> 42.0 mm
- net Net-(CON3-Pad3): track 0.00 -> 11.6 mm
- net Net-(CON2-Pad3): track 0.00 -> 9.04 mm
- net /~EF3: track 25.4 -> 19.7 mm
- net Net-(CON3-Pad4): track 0.00 -> 3.17 mm
- net VCC: track 162.6 -> 160.9 mm
- net /MA7: track 49.7 -> 50.8 mm
- net /BUS7: track 13.0 -> 13.7 mm
- net Net-(CON2-Pad4): track 11.4 -> 12.1 mm
Other:
- board text added: "2022/06/25 @kanpapa"
- board text added: "EMU1802-mini Rev. 1.0"
- board text removed: "EMU1802-mini Rev. 0.1 2022/06/11 @kanpapa"
