File: kicad/emu1802_mini/emu1802_mini.kicad_sch (KiCad schematic)
At the start: 21 parts, among them CON1 PICKIT/SNAP, CON2 UART, CON3 Software Serial, CON4 DC-IN, J1 CPUA, J2 CPUB, SW1 POWER, SW2 RESET, U1 CDP1802ACE, U2 PIC18F27Q43

Commit message: Updated emu1802-mini PCB Rev.1.0
Parts:
- added D2: 1N4148, Diode_THT:D_T-1_P5.08mm_Horizontal, symbol Device:D
- added JP1: BUS POWER1, Jumper:SolderJumper-2_P1.3mm_Open_RoundedPad1.0x1.5mm, symbol Jumper:SolderJumper_2_Open
- added JP2: BUS POWER2, Jumper:SolderJumper-2_P1.3mm_Open_RoundedPad1.0x1.5mm, symbol Jumper:SolderJumper_2_Open
Connections:
- net ~EF3: now also D2.2 (A); no longer CON3.4 (Pin_4)
- net +5V: now reaches CON4.1 (Pin_1), SW1.3 (C)
- net +5V: now also JP1.2 (B), JP2.2 (B)
- net at CON2.3 (Pin_3): now also JP1.1 (A)
- net at CON3.3 (Pin_3): now also JP2.1 (A)
- new net: CON3.4 (Pin_4), D2.1 (K)
- no-connect marks 10 -> 8
Other:
- note added: "Vcc"
